File: Project/Khanh_eagleProject/firstProject/firstProject_1.1/firstProject_1.1.brd (EAGLE design)
At the start: 40 x 12 mm, 13 parts

Commit message: update ams1117 5v v1.1
Routing:
- net N$3: track 51.4 -> 49.5 mm
- removed copper zone on layer 1, net N$1
